File: CheerLights1Channel.sch (EAGLE design)
At the start: 9 parts, among them J1 GREEN-3P-5.0, J2 DC-005, J3 GREEN-2P-3.5

Commit message: Add files via upload
Updated schematic and board files
Parts:
- removed FRAME1: FRAME-LETTER, Mawrey:FRAME-LETTER
- renumbered U$1 to U1, U$2 to U2
Connections:
- net GND: now also U1.GND@21
Changed lines of the file:
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@@
 </classes>
 <parts>
-<part name="U$1" library="Particle" deviceset="PHOTON" device="_WITH_HEADERS"/>
-<part name="U$2" library="Mawrey" deviceset="BUFFER" device="SN74LV1T34"/>
+<part name="U1" library="Particle" deviceset="PHOTON" device="_WITH_HEADERS"/>
+<part name="U2" library="Mawrey" deviceset="BUFFER" device="SN74LV1T34"/>
 <part name="GND1" library="Mawrey" deviceset="GND" device=""/>
 <part name="SUPPLY1" library="SparkFun-Aesthetics" deviceset="5V" device=""/>
-<part name="FRAME1" library="Mawrey" deviceset="FRAME-LETTER" device=""/>
 <part name="J1" library="Seeed-Connector -2016" deviceset="SCREW-TERMINAL-GREEN(3P-5.0)" device="" value="GREEN-3P-5.0">
 <attribute name="PARTNO" value="1935174"/>
@@
 <part name="SUPPLY5" library="SparkFun-Aesthetics" deviceset="5V" device=""/>
 <part name="C1" library="Mawrey" deviceset="CAP" device="0805" value="0.1uF"/>
-<part name="U$3" library="Mawrey" deviceset="0805_CAP" device=""/>
 <part name="C3" library="Mawrey" deviceset="CAP" device="0805" value="1uF"/>
 <part name="GND7" library="Mawrey" deviceset="GND" device=""/>
@@
 <part name="SUPPLY7" library="SparkFun-Aesthetics" deviceset="5V" device=""/>
 <part name="SUPPLY8" library="SparkFun-Aesthetics" deviceset="5V" device=""/>
+<part name="GND6" library="Mawrey" deviceset="GND" device=""/>
 </parts>
 <sheets>
@@
 </plain>
 <instances>
-<instance part="U$1" gate="G$1" x="100.33" y="107.95"/>
-<instance part="U$2" gate="G$1" x="138.43" y="80.01"/>
+<instance part="U1" gate="G$1" x="100.33" y="107.95"/>
+<instance part="U2" gate="G$1" x="138.43" y="80.01"/>
 <instance part="GND1" gate="1" x="138.43" y="68.58"/>
 <instance part="SUPPLY1" gate="G$1" x="138.43" y="90.17"/>
-<instance part="FRAME1" gate="G$1" x="0" y="0"/>
-<instance part="FRAME1" gate="V" x="147.32" y="0"/>
 <instance part="J1" gate="G$1" x="176.53" y="80.01">
 <attribute name="PARTNO" x="176.53" y="80.01" size="1.778" layer="96" rot="R270" display="off"/>
@@
 <instance part="SUPPLY7" gate="G$1" x="148.59" y="134.62"/>
 <instance part="SUPPLY8" gate="G$1" x="157.48" y="134.62"/>
+<instance part="GND6" gate="1" x="123.19" y="115.57"/>
 </instances>
 <busses>
@@
 <net name="DATA" class="0">
 <segment>
-<pinref part="U$1" gate="G$1" pin="D0"/>
-<pinref part="U$2" gate="G$1" pin="IN"/>
+<pinref part="U1" gate="G$1" pin="D0"/>
+<pinref part="U2" gate="G$1" pin="IN"/>
 <wire x1="133.35" y1="80.01" x2="118.11" y2="80.01" width="0.1524" layer="91"/>
 </segment>
@@
 <net name="GND" class="1">
 <segment>
-<pinref part="U$2" gate="G$1" pin="GND"/>
+<pinref part="U2" gate="G$1" pin="GND"/>
 <pinref part="GND1" gate="1" pin="GND"/>
 <wire x1="138.43" y1="71.12" x2="138.43" y2="74.93" width="0.1524" layer="91"/>
 </segment>
 <segment>
-<pinref part="U$1" gate="G$1" pin="GND@2"/>
+<pinref part="U1" gate="G$1" pin="GND@2"/>
 <pinref part="J2" gate="JACK" pin="-"/>
 <wire x1="69.85" y1="130.81" x2="82.55" y2="130.81" width="0.1524" layer="91"/>
@@
 <wire x1="157.48" y1="123.19" x2="157.48" y2="124.46" width="0.1524" layer="91"/>
 </segment>
+<segment>
+<pinref part="U1" gate="G$1" pin="GND@21"/>
+<pinref part="GND6" gate="1" pin="GND"/>
+<wire x1="118.11" y1="120.65" x2="123.19" y2="120.65" width="0.1524" layer="91"/>
+<wire x1="123.19" y1="120.65" x2="123.19" y2="118.11" width="0.1524" layer="91"/>
+</segment>
 </net>
 <net name="5V" class="1">
 <segment>
-<pinref part="U$2" gate="G$1" pin="PWR"/>
+<pinref part="U2" gate="G$1" pin="PWR"/>
 <pinref part="SUPPLY1" gate="G$1" pin="5V"/>
 <wire x1="138.43" y1="90.17" x2="138.43" y2="85.09" width="0.1524" layer="91"/>
 </segment>
 <segment>
-<pinref part="U$1" gate="G$1" pin="VIN"/>
+<pinref part="U1" gate="G$1" pin="VIN"/>
 <pinref part="J2" gate="JACK" pin="+"/>
 <wire x1="69.85" y1="135.89" x2="82.55" y2="135.89" width="0.1524" layer="91"/>
@@
 <segment>
 <pinref part="J1" gate="G$1" pin="P$2"/>
-<pinref part="U$2" gate="G$1" pin="OUT"/>
+<pinref part="U2" gate="G$1" pin="OUT"/>
 <wire x1="168.91" y1="80.01" x2="157.48" y2="80.01" width="0.1524" layer="91"/>
 <pinref part="D2" gate="G$1" pin="1"/>
