File: CheerLights1Channel.brd (EAGLE design)
At the start: 38.1 x 20.3 mm, 9 parts, among them J1 GREEN-3P-5.0, J2 DC-005, J3 GREEN-2P-3.5

Commit message: Add files via upload
Updated schematic and board files
Parts:
- removed FRAME1: FRAME-LETTER, Mawrey:CREATIVE_COMMONS
- moved C3 9.55 mm to (15.7, 4.57)
- moved C1 8.92 mm to (15.7, 3.30)
- moved J3 3.81 mm to (10.2, 5.71)
- renumbered U$1 to U1, U$2 to U2
Routing:
- net 5V: track 31.3 -> 27.5 mm
- net GND: track 2.37 -> 5.89 mm
- net DOUT: track 14.8 -> 16.0 mm

Commit message: Add files via upload
Lastest versions
Parts:
- moved C3 1.27 mm to (15.8, 3.30)
- moved C1 1.27 mm to (15.8, 4.57)
Routing:
- net 5V: track 27.5 -> 25.9 mm, vias 1 -> 0
- net DATA: track 21.4 -> 19.8 mm
- net DOUT: track 16.0 -> 14.7 mm
